File: Tester/Tester.kicad_pcb (KiCad board)
At the start: 4 copper layers, 100 x 100 mm, 58 parts, among them J1 Conn_Coaxial, J2 Conn_Coaxial, J3 Conn_Coaxial, J4 Conn_Coaxial, J5 Conn_Coaxial, J6 Conn_Coaxial, J7 Conn_02x12_Counter_Clockwise, J8 Conn_01x03_Female, J9 Conn_01x03_Female, SW1 SW_Rotary2x6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

Commit message: routing
Parts:
- moved D2 19.5 mm to (92.0, 115.5)
- moved JP2 8.72 mm to (121.8, 145.0)
- moved R23 8.55 mm to (103.5, 76.5), turned to 180 degrees
- moved R26 8.51 mm to (122.0, 145.0)
- moved D4 4.00 mm to (137.5, 145.0)
- moved R24 2.50 mm to (103.0, 118.5)
Routing:
- net /DUT11: track 0.00 -> 121.1 mm
- net /DUT12: track 0.00 -> 111.3 mm
- net /DUT21: track 0.00 -> 105.2 mm
- net /DUT23: track 0.00 -> 101.3 mm
- net /I2: track 0.00 -> 97.0 mm, vias 0 -> 3
- net /DUT13: track 0.00 -> 94.1 mm
- net Net-(R14-Pad1): track 0.00 -> 84.0 mm
- net /V2: track 19.1 -> 100.1 mm, vias 0 -> 3
- net /DUT22: track 0.00 -> 79.3 mm
- net Net-(R17-Pad1): track 0.00 -> 75.5 mm
- net /V1: track 24.8 -> 99.4 mm, vias 0 -> 1
- net Net-(R3-Pad1): track 0.00 -> 71.6 mm
- net Net-(R16-Pad1): track 0.00 -> 70.1 mm
- net Net-(R2-Pad1): track 0.00 -> 59.9 mm
- net Net-(R10-Pad1): track 0.00 -> 55.1 mm
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- removed copper zone on InB.Cu, net /I1
- removed copper zone on InF.Cu, net /I2
